Commit message: Fix camera in dockerfile

File: xavbot_description/urdf/xavbot.xacro (robot description, xacro)
@@ -52,5 +52,5 @@
       </collision>
       <visual>
-        <origin xyz="0 0 0" rpy="0 0 0"/>
+        <origin xyz="0 0 0" rpy="${PI} 0 0"/>
         <geometry>
           <mesh filename="package://xavbot_description/meshes/d435.stl" scale="0.001 0.001 0.001"/>
@@ -62,5 +62,5 @@
       <parent link="${prefix}chassis_link"/>
       <child link="${prefix}camera_link"/>
-      <origin xyz="0.085 0 0.028" rpy="0 0 0"/>
+      <origin xyz="0.085 0 0.028" rpy="${PI} 0 0"/>
     </joint>
     <!-- front left wheel link -->

Commit message: add base_footprint

File: xavbot_description/urdf/xavbot.xacro (robot description, xacro)
@@ -13,7 +13,4 @@
   <!-- Base Link -->
   <link name="${prefix}base_link">
-  </link>
-  <!-- Chassis Link -->
-  <link name="${prefix}chassis_link">
     <collision>
       <origin xyz="0 0 ${base_height/2}" rpy="0 0 0"/>
@@ -38,8 +35,10 @@
       </inertial>
     </link>
+    <!-- Base Footprint -->
+    <link name="${prefix}base_footprint"></link>
     <joint name="${prefix}chassis_joint" type="fixed">
       <parent link="${prefix}base_link"/>
-      <child link="${prefix}chassis_link"/>
-      <origin xyz="0 0 ${wheel_radius}" rpy="0 0 0"/>
+      <child link="${prefix}base_footprint"/>
+      <origin xyz="0 0 ${-wheel_radius}" rpy="0 0 0"/>
     </joint>
     <!-- Camera Link -->
@@ -60,5 +59,5 @@
     </link>
     <joint name="${prefix}camera_joint" type="fixed">
-      <parent link="${prefix}chassis_link"/>
+      <parent link="${prefix}base_link"/>
       <child link="${prefix}camera_link"/>
       <origin xyz="0.085 0 0.028" rpy="${PI} 0 0"/>
@@ -66,5 +65,5 @@
     <!-- front left wheel link -->
     <joint name="${prefix}front_left_wheel_joint" type="continuous">
-      <parent link="${prefix}chassis_link"/>
+      <parent link="${prefix}base_link"/>
       <child link="${prefix}front_left_wheel"/>
       <origin xyz="${base_length/2} ${(base_width + wheel_length)/2} 0" rpy="0 0 0"/>
@@ -97,5 +96,5 @@
     <!-- front right wheel link -->
     <joint name="${prefix}front_right_wheel_joint" type="continuous">
-      <parent link="${prefix}chassis_link"/>
+      <parent link="${prefix}base_link"/>
       <child link="${prefix}front_right_wheel"/>
       <origin xyz="${base_length/2} -${(base_width + wheel_length)/2} 0" rpy="0 0 0"/>
@@ -128,5 +127,5 @@
       <!-- rear left wheel link -->
       <joint name="${prefix}rear_left_wheel_joint" type="continuous">
-        <parent link="${prefix}chassis_link"/>
+        <parent link="${prefix}base_link"/>
         <child link="${prefix}rear_left_wheel"/>
         <origin xyz="-${base_length/2} ${(base_width + wheel_length)/2} 0" rpy="0 0 0"/>
@@ -159,5 +158,5 @@
       <!-- rear right wheel link -->
       <joint name="${prefix}rear_right_wheel_joint" type="continuous">
-        <parent link="${prefix}chassis_link"/>
+        <parent link="${prefix}base_link"/>
         <child link="${prefix}rear_right_wheel"/>
         <origin xyz="-${base_length/2} -${(base_width + wheel_length)/2} 0" rpy="0 0 0"/>
