Commit message: URDF updates

File: xavbot_description/urdf/xavbot.arm.xacro (robot description, xacro)
@@ -8,5 +8,5 @@
         <parent link="${prefix}base_link"/>
         <child link="${prefix}link0"/>
-        <origin xyz="0.21575 0.185 0.068" rpy="${PI/2} 0 0"/>
+        <origin xyz="0.210 0.200 0.073" rpy="${PI/2} 0 0"/>
         <axis xyz="0 0 0"/>
         <dynamics damping="0.2"/>
@@ -19,10 +19,10 @@
       </joint>
       <link name="${prefix}link0">
-        <!-- <collision>
-          <origin xyz="0 0 0.05" rpy="0 0 0"/>
+        <collision>
+          <origin xyz="0 -0.013 0" rpy="0 0 0"/>
           <geometry>
-            <mesh filename="${mesh_dir}/collision/link0.stl" scale="0.001 0.001 0.001"/>
+            <box size="0.0285 0.0465 0.034"/>
           </geometry>
-        </collision> -->
+        </collision>
         <visual>
           <origin xyz="0 0 0" rpy="0 0 0"/>
@@ -32,4 +32,12 @@
           <material name="grey"/>
         </visual>
+        <inertial>
+          <origin xyz="0 -0.013 0" rpy="0 0 0"/>
+          <mass value="0.0572"/>
+          <inertia
+            ixx="${0.0572 / 12.0 * (0.0465*0.0465 + 0.034*0.034)}" ixy="0.0" ixz="0.0"
+            iyy="${0.0572 / 12.0 * (0.034*0.034 + 0.0285*0.0285)}" iyz="0.0"
+            izz="${0.0572 / 12.0 * (0.0285*0.0285 + 0.0465*0.0465)}"/>
+        </inertial>
       </link>
       <!-- link1 -->
@@ -48,10 +56,10 @@
       </joint>
       <link name="${prefix}link1">
-        <!-- <collision>
-          <origin xyz="0 0 0.05" rpy="0 0 0"/>
+        <collision>
+          <origin xyz="0 0.140 0" rpy="0 0 0"/>
           <geometry>
-            <box size="0.02 0.02 0.1"/>
+            <box size="0.0285 0.140 0.034"/>
           </geometry>
-        </collision> -->
+        </collision>
         <visual>
           <origin xyz="0 0 0" rpy="0 0 0"/>
@@ -61,4 +69,12 @@
           <material name="grey"/>
         </visual>
+        <inertial>
+          <origin xyz="0 -0.013 0" rpy="0 0 0"/>
+          <mass value="0.0572"/>
+          <inertia
+            ixx="${0.0572 / 12.0 * (0.0465*0.0465 + 0.034*0.034)}" ixy="0.0" ixz="0.0"
+            iyy="${0.0572 / 12.0 * (0.034*0.034 + 0.0285*0.0285)}" iyz="0.0"
+            izz="${0.0572 / 12.0 * (0.0285*0.0285 + 0.0465*0.0465)}"/>
+        </inertial>
       </link>
       <!-- link2 -->
@@ -71,5 +87,5 @@
         <limit
           lower="-${PI/2}"
-          upper="${PI/2}"
+          upper="${3 * PI/4}"
           effort="4"
           velocity="4.5">
@@ -95,10 +111,10 @@
         <parent link="${prefix}link2"/>
         <child link="${prefix}link3"/>
-        <origin xyz="0.130 0.038 0" rpy="0 0 -${PI/2}"/>
+        <origin xyz="0.1 0.04 0" rpy="0 0 -${PI/2}"/>
         <axis xyz="0 0 1 "/>
         <dynamics damping="0.2"/>
         <limit
           lower="-${PI/2}"
-          upper="${3 * PI/4}"
+          upper="${PI/2}"
           effort="4"
           velocity="4.5">
@@ -124,5 +140,5 @@
         <parent link="${prefix}link3"/>
         <child link="${prefix}link4"/>
-        <origin xyz="0 0.043 -0.012" rpy="${PI/2} 0 ${PI/2}"/>
+        <origin xyz="0 0.061 0" rpy="${-PI/2} ${PI/2} 0"/>
         <axis xyz="0 0 1"/>
         <dynamics damping="0.2"/>
@@ -153,5 +169,5 @@
         <parent link="${prefix}link4"/>
         <child link="${prefix}tool0"/>
-        <origin xyz="0 0 0.08" rpy="0 ${-PI/2} 0"/>
+        <origin xyz="0 0 0.08" rpy="${PI/2} ${-PI/2} 0"/>
       </joint>
       <link name="${prefix}tool0"/>

File: xavbot_description/urdf/xavbot.platform.xacro (robot description, xacro)
@@ -5,6 +5,6 @@
   <xacro:property name="PI" value="3.1415926535897931"/>
   <xacro:property name="base_mass" value="1.0" /> <!-- arbitrary value for base mass -->
-  <xacro:property name="base_width" value="0.11" />
-  <xacro:property name="base_length" value="0.12" />
+  <xacro:property name="base_width" value="0.25" />
+  <xacro:property name="base_length" value="0.25" />
   <xacro:property name="base_height" value="0.05" />
   <xacro:property name="wheel_mass" value="0.02" /> <!-- arbitrary value for wheel mass -->
@@ -15,5 +15,5 @@
   <link name="${prefix}base_link">
     <collision>
-      <origin xyz="0.125 0.125 ${wheel_radius + 0.04}" rpy="0 0 0"/>
+      <origin xyz="${base_width / 2} ${base_length / 2} ${wheel_radius + 0.04}" rpy="0 0 0"/>
       <geometry>
         <box size="0.25 0.25 0.08"/>
@@ -28,5 +28,5 @@
     </visual>
     <inertial>
-      <origin xyz="0 0 ${wheel_radius + 0.04}" rpy="0 0 0"/>
+      <origin xyz="${base_width / 2} ${base_length / 2} ${wheel_radius + base_height / 2}" rpy="0 0 0"/>
       <mass value="${base_mass}"/>
       <inertia

Commit message: Initial arm setup

File: xavbot_description/urdf/xavbot.arm.xacro (robot description, xacro)
@@ -1,26 +1,44 @@
 <?xml version="1.0"?>
 <robot xmlns:xacro="http://www.ros.org/wiki/xacro" name="xavbot">
-  <xacro:macro name="xavbot_arm" params="prefix='' mesh_dir='package://xavbot_description/meshes'">
+  <xacro:macro name="xavbot_arm" params="prefix='' mesh_dir='package://xavbot_description/meshes' standalone='true'">
   <!-- Constants for robot dimensions -->
   <xacro:property name="PI" value="3.1415926535897931"/>
-        <!-- link0 -->
-      <joint name="${prefix}link0_joint" type="fixed">
-        <parent link="${prefix}base_link"/>
-        <child link="${prefix}link0"/>
-        <origin xyz="0.210 0.200 0.073" rpy="${PI/2} 0 0"/>
-        <axis xyz="0 0 0"/>
-        <dynamics damping="0.2"/>
-        <limit
-          lower="-${PI/4}"
-          upper="${PI/2}"
-          effort="4"
-          velocity="4.5">
-        </limit>
-      </joint>
+      <!-- link0 -->
+      <xacro:if value="${standalone}">
+        <link name="${prefix}base_link" />
+        <joint name="${prefix}link0_joint" type="fixed">
+          <parent link="${prefix}base_link"/>
+          <child link="${prefix}link0"/>
+          <origin xyz="0 0 0" rpy="${PI/2} 0 0"/>
+          <axis xyz="0 0 0"/>
+          <dynamics damping="0.2"/>
+          <limit
+            lower="-${PI/2}"
+            upper="${PI/2}"
+            effort="4"
+            velocity="6">
+          </limit>
+        </joint>
+      </xacro:if>
+      <xacro:unless value="${standalone}">
+        <joint name="${prefix}link0_joint" type="fixed">
+          <parent link="${prefix}base_link"/>
+          <child link="${prefix}link0"/>
+          <origin xyz="0.210 0.200 0.073" rpy="${PI/2} 0 0"/>
+          <axis xyz="0 0 0"/>
+          <dynamics damping="0.2"/>
+          <limit
+            lower="-${PI/2}"
+            upper="${PI/2}"
+            effort="4"
+            velocity="6">
+          </limit>
+        </joint>
+      </xacro:unless>
       <link name="${prefix}link0">
         <collision>
-          <origin xyz="0 -0.013 0" rpy="0 0 0"/>
+          <origin xyz="0 0 0" rpy="0 0 0"/>
           <geometry>
-            <box size="0.0285 0.0465 0.034"/>
+            <mesh filename="${mesh_dir}/collision/link0.stl" scale="0.001 0.001 0.001"/>
           </geometry>
         </collision>
@@ -46,18 +64,18 @@
         <child link="${prefix}link1"/>
         <origin xyz="0 0 0" rpy="0 0 0"/>
-        <axis xyz="0 0 1"/>
+        <axis xyz="0 0 -1"/>
         <dynamics damping="0.2"/>
         <limit
-          lower="-${PI/2}"
-          upper="${PI/2}"
+          lower="${PI/2}"
+          upper="${3* PI/2}"
           effort="4"
-          velocity="4.5">
+          velocity="6">
         </limit>
       </joint>
       <link name="${prefix}link1">
         <collision>
-          <origin xyz="0 0.140 0" rpy="0 0 0"/>
+          <origin xyz="0 0 0" rpy="0 0 0"/>
           <geometry>
-            <box size="0.0285 0.140 0.034"/>
+            <mesh filename="${mesh_dir}/collision/link1.stl" scale="0.001 0.001 0.001"/>
           </geometry>
         </collision>
@@ -83,20 +101,20 @@
         <child link="${prefix}link2"/>
         <origin xyz="0 0.1 0" rpy="0 0 0"/>
-        <axis xyz="0 0 1"/>
+        <axis xyz="0 0 -1"/>
         <dynamics damping="0.2"/>
         <limit
-          lower="-${PI/2}"
-          upper="${3 * PI/4}"
+          lower="${PI/9}"
+          upper="${3 * PI/2}"
           effort="4"
-          velocity="4.5">
+          velocity="6">
         </limit>
       </joint>
       <link name="${prefix}link2">
-        <!-- <collision>
-          <origin xyz="0 0 0.015" rpy="0 0 0"/>
+        <collision>
+          <origin xyz="0 0 0" rpy="0 0 0"/>
           <geometry>
-            <box size="0.02 0.02 0.03"/>
+            <mesh filename="${mesh_dir}/collision/link2.stl" scale="0.001 0.001 0.001"/>
           </geometry>
-        </collision> -->
+        </collision>
         <visual>
           <origin xyz="0 0 0" rpy="0 0 0"/>
@@ -111,21 +129,21 @@
         <parent link="${prefix}link2"/>
         <child link="${prefix}link3"/>
-        <origin xyz="0.1 0.04 0" rpy="0 0 -${PI/2}"/>
-        <axis xyz="0 0 1 "/>
+        <origin xyz="0.1 0.04 0" rpy="0 0 ${-PI/2}"/>
+        <axis xyz="0 0 -1 "/>
         <dynamics damping="0.2"/>
         <limit
-          lower="-${PI/2}"
-          upper="${PI/2}"
+          lower="${PI/2}"
+          upper="${3 * PI/2}"
           effort="4"
-          velocity="4.5">
+          velocity="6">
         </limit>
       </joint>
       <link name="${prefix}link3">
-        <!-- <collision>
-          <origin xyz="0 0 0.015" rpy="0 0 0"/>
+        <collision>
+          <origin xyz="0 0 0" rpy="0 0 0"/>
           <geometry>
-            <box size="0.02 0.02 0.03"/>
+            <mesh filename="${mesh_dir}/collision/link3.stl" scale="0.001 0.001 0.001"/>
           </geometry>
-        </collision> -->
+        </collision>
         <visual>
           <origin xyz="0 0 0" rpy="0 0 0"/>
@@ -147,14 +165,14 @@
           upper="${PI}"
           effort="4"
-          velocity="4.5">
+          velocity="6">
         </limit>
       </joint>
       <link name="${prefix}link4">
-        <!-- <collision>
-          <origin xyz="0 0 0.015" rpy="0 0 0"/>
+        <collision>
+          <origin xyz="0 0 0" rpy="0 0 0"/>
           <geometry>
-            <box size="0.02 0.02 0.03"/>
+            <mesh filename="${mesh_dir}/collision/link4.stl" scale="0.001 0.001 0.001"/>
           </geometry>
-        </collision> -->
+        </collision>
         <visual>
           <origin xyz="0 0 0" rpy="0 0 0"/>

File: xavbot_description/urdf/xavbot.platform.ros2_control.xacro (robot description, xacro)
@@ -1,5 +1,5 @@
 <?xml version="1.0"?>
 <robot xmlns:xacro="http://www.ros.org/wiki/xacro">
-  <xacro:macro name="xavbot_ros2_control" params="name prefix">
+  <xacro:macro name="xavbot_platform_control" params="name prefix">
     <ros2_control name="${name}" type="system">
       <hardware>

File: xavbot_description/urdf/xavbot.platform.xacro (robot description, xacro)
@@ -1,5 +1,5 @@
 <?xml version="1.0"?>
 <robot xmlns:xacro="http://www.ros.org/wiki/xacro" name="xavbot">
-  <xacro:macro name="xavbot_platform" params="prefix='' mesh_dir='package://xavbot_description/meshes'">
+  <xacro:macro name="xavbot_platform" params="prefix='' mesh_dir='package://xavbot_description/meshes' ">
   <!-- Constants for robot dimensions -->
   <xacro:property name="PI" value="3.1415926535897931"/>

File: xavbot_description/urdf/xavbot.urdf.xacro (robot description, xacro)
@@ -2,13 +2,21 @@
 <robot xmlns:xacro="http://www.ros.org/wiki/xacro" name="xavbot">
   <xacro:arg name="prefix" default="" />
+  <xacro:arg name="arm" default="true" />
   <!-- Import Geometry -->
   <xacro:include filename="$(find xavbot_description)/urdf/xavbot.platform.xacro" />
   <xacro:xavbot_platform prefix="$(arg prefix)" mesh_dir="package://xavbot_description/meshes" />
-  <xacro:include filename="$(find xavbot_description)/urdf/xavbot.arm.xacro" />
-  <xacro:xavbot_arm prefix="$(arg prefix)" mesh_dir="package://xavbot_description/meshes" />
+  <!-- Import xavbot ros2_control description -->
+  <xacro:include filename="$(find xavbot_description)/urdf/xavbot.platform.ros2_control.xacro" />
+  <xacro:xavbot_platform_control name="xavbot" prefix="$(arg prefix)" />
   <!-- Import Rviz colors -->
   <xacro:include filename="$(find xavbot_description)/urdf/xavbot.materials.xacro" />
-  <!-- Import xavbot ros2_control description -->
-  <xacro:include filename="$(find xavbot_description)/urdf/xavbot.ros2_control.xacro" />
-  <xacro:xavbot_ros2_control name="xavbot" prefix="$(arg prefix)" />
+  <!-- Import xavbot_arm -->
+  <xacro:if value="$(arg arm)">
+    <!-- Import Geometry -->
+    <xacro:include filename="$(find xavbot_description)/urdf/xavbot.arm.xacro" />
+    <xacro:xavbot_arm prefix="$(arg prefix)" mesh_dir="package://xavbot_description/meshes" standalone="false" />
+    <!-- Import xavbot ros2_control description -->
+    <xacro:include filename="$(find xavbot_description)/urdf/xavbot.arm.ros2_control.xacro" />
+    <xacro:xavbot_arm_control name="xavbot" prefix="$(arg prefix)" />
+  </xacro:if>
 </robot>
