Commit message: moveit config

File: xavbot_description/urdf/xavbot.arm.ros2_control.xacro (robot description, xacro)
@@ -10,4 +10,5 @@
       <joint name="${prefix}link1_joint">
         <param name="id">10</param>
+        <param name="offset">3.141592</param>
         <command_interface name="position"/>
         <command_interface name="velocity"/>
@@ -18,4 +19,5 @@
       <joint name="${prefix}link2_joint">
         <param name="id">11</param>
+        <param name="offset">3.141592</param>
         <command_interface name="position"/>
         <command_interface name="velocity"/>
@@ -26,4 +28,5 @@
       <joint name="${prefix}link3_joint">
         <param name="id">12</param>
+        <param name="offset">3.141592</param>
         <command_interface name="position"/>
         <command_interface name="velocity"/>
@@ -34,4 +37,5 @@
       <joint name="${prefix}link4_joint">
         <param name="id">13</param>
+        <param name="offset">3.141592</param>
         <command_interface name="position"/>
         <command_interface name="velocity"/>

File: xavbot_description/urdf/xavbot.arm.xacro (robot description, xacro)
@@ -10,13 +10,5 @@
           <parent link="${prefix}base_link"/>
           <child link="${prefix}link0"/>
-          <origin xyz="0 0 0" rpy="${PI/2} 0 0"/>
-          <axis xyz="0 0 0"/>
-          <dynamics damping="0.2"/>
-          <limit
-            lower="-${PI/2}"
-            upper="${PI/2}"
-            effort="4"
-            velocity="6">
-          </limit>
+          <origin xyz="0 0 0" rpy="${PI/2} 0 ${PI}"/>
         </joint>
       </xacro:if>
@@ -25,13 +17,5 @@
           <parent link="${prefix}base_link"/>
           <child link="${prefix}link0"/>
-          <origin xyz="0.210 0.200 0.073" rpy="${PI/2} 0 0"/>
-          <axis xyz="0 0 0"/>
-          <dynamics damping="0.2"/>
-          <limit
-            lower="-${PI/2}"
-            upper="${PI/2}"
-            effort="4"
-            velocity="6">
-          </limit>
+          <origin xyz="0.210 0.200 0.073" rpy="${PI/2} 0 ${PI}"/>
         </joint>
       </xacro:unless>
@@ -64,11 +48,11 @@
         <child link="${prefix}link1"/>
         <origin xyz="0 0 0" rpy="0 0 0"/>
-        <axis xyz="0 0 -1"/>
+        <axis xyz="0 0 1"/>
         <dynamics damping="0.2"/>
         <limit
-          lower="${PI/2}"
-          upper="${3* PI/2}"
-          effort="4"
-          velocity="6">
+          lower="${-PI/2}"
+          upper="${PI/2}"
+          effort="4.0"
+          velocity="6.1">
         </limit>
       </joint>
@@ -101,11 +85,11 @@
         <child link="${prefix}link2"/>
         <origin xyz="0 0.1 0" rpy="0 0 0"/>
-        <axis xyz="0 0 -1"/>
+        <axis xyz="0 0 1"/>
         <dynamics damping="0.2"/>
         <limit
-          lower="${PI/9}"
-          upper="${3 * PI/2}"
-          effort="4"
-          velocity="6">
+          lower="${-8 * PI/9}"
+          upper="${PI/2}"
+          effort="4.0"
+          velocity="6.1">
         </limit>
       </joint>
@@ -129,12 +113,12 @@
         <parent link="${prefix}link2"/>
         <child link="${prefix}link3"/>
-        <origin xyz="0.1 0.04 0" rpy="0 0 ${-PI/2}"/>
-        <axis xyz="0 0 -1 "/>
+        <origin xyz="-0.1 0.04 0" rpy="0 0 0"/>
+        <axis xyz="0 0 1 "/>
         <dynamics damping="0.2"/>
         <limit
-          lower="${PI/2}"
-          upper="${3 * PI/2}"
-          effort="4"
-          velocity="6">
+          lower="${-PI/2}"
+          upper="${PI/2}"
+          effort="4.0"
+          velocity="6.1">
         </limit>
       </joint>
@@ -158,5 +142,5 @@
         <parent link="${prefix}link3"/>
         <child link="${prefix}link4"/>
-        <origin xyz="0 0.061 0" rpy="${-PI/2} ${PI/2} 0"/>
+        <origin xyz="-0.061 0 0" rpy="0 ${-PI/2} 0"/>
         <axis xyz="0 0 1"/>
         <dynamics damping="0.2"/>
@@ -164,6 +148,6 @@
           lower="-${PI}"
           upper="${PI}"
-          effort="4"
-          velocity="6">
+          effort="4.0"
+          velocity="6.1">
         </limit>
       </joint>

Commit message: Add and configure gripper

File: xavbot_description/urdf/xavbot.arm.ros2_control.xacro (robot description, xacro)
@@ -10,5 +10,4 @@
       <joint name="${prefix}link1_joint">
         <param name="id">10</param>
-        <param name="offset">3.141592</param>
         <command_interface name="position"/>
         <command_interface name="velocity"/>
@@ -19,5 +18,4 @@
       <joint name="${prefix}link2_joint">
         <param name="id">11</param>
-        <param name="offset">3.141592</param>
         <command_interface name="position"/>
         <command_interface name="velocity"/>
@@ -28,5 +26,4 @@
       <joint name="${prefix}link3_joint">
         <param name="id">12</param>
-        <param name="offset">3.141592</param>
         <command_interface name="position"/>
         <command_interface name="velocity"/>
@@ -37,5 +34,12 @@
       <joint name="${prefix}link4_joint">
         <param name="id">13</param>
-        <param name="offset">3.141592</param>
+        <command_interface name="position"/>
+        <command_interface name="velocity"/>
+        <state_interface name="position"/>
+        <state_interface name="velocity"/>
+        <state_interface name="effort"/>
+      </joint>
+      <joint name="${prefix}gripper_joint">
+        <param name="id">14</param>
         <command_interface name="position"/>
         <command_interface name="velocity"/>

File: xavbot_description/urdf/xavbot.arm.xacro (robot description, xacro)
@@ -54,5 +54,5 @@
           upper="${PI/2}"
           effort="4.0"
-          velocity="6.1">
+          velocity="5.5">
         </limit>
       </joint>
@@ -91,5 +91,5 @@
           upper="${PI/2}"
           effort="4.0"
-          velocity="6.1">
+          velocity="5.5">
         </limit>
       </joint>
@@ -120,5 +120,5 @@
           upper="${PI/2}"
           effort="4.0"
-          velocity="6.1">
+          velocity="5.5">
         </limit>
       </joint>
@@ -149,5 +149,5 @@
           upper="${PI}"
           effort="4.0"
-          velocity="6.1">
+          velocity="5.5">
         </limit>
       </joint>
@@ -167,11 +167,83 @@
         </visual>
       </link>
-      <!-- tool0 -->
-      <joint name="${prefix}tool0_joint" type="fixed">
-        <parent link="${prefix}link4"/>
-        <child link="${prefix}tool0"/>
+      <!-- hand_tcp -->
+      <joint name="${prefix}tcp_joint" type="fixed">
+        <parent link="${prefix}link4"/>
+        <child link="${prefix}tcp"/>
         <origin xyz="0 0 0.08" rpy="${PI/2} ${-PI/2} 0"/>
       </joint>
-      <link name="${prefix}tool0"/>
+      <link name="${prefix}tcp"/>
+      <!-- gripper_crank -->
+      <joint name="${prefix}gripper_joint" type="revolute">
+        <parent link="${prefix}link4"/>
+        <child link="${prefix}gripper_crank"/>
+        <origin xyz="0 0 0.04" rpy="0 0 0"/>
+        <axis xyz="0 0 1"/>
+        <limit
+          lower="0"
+          upper="1.047"
+          effort="4.0"
+          velocity="5.5">
+        </limit>
+      </joint>
+      <link name="${prefix}gripper_crank"/>
+      <!-- rightfinger -->
+      <joint name="${prefix}rightfinger_joint" type="prismatic">
+        <parent link="${prefix}link4"/>
+        <child link="${prefix}rightfinger"/>
+        <origin xyz="0 0 0.045" rpy="0 0 0"/>
+        <axis xyz="-1 0 0"/>
+        <limit
+          lower="0"
+          upper="0.0265"
+          effort="9.9"
+          velocity="9.9">
+        </limit>
+        <mimic joint="${prefix}gripper_joint" multiplier="0.024446"/>
+      </joint>
+      <link name="${prefix}rightfinger">
+        <collision>
+          <origin xyz="0 0 0" rpy="0 0 0"/>
+          <geometry>
+            <mesh filename="${mesh_dir}/collision/finger.stl" scale="0.001 0.001 0.001"/>
+          </geometry>
+        </collision>
+        <visual>
+          <origin xyz="0 0 0" rpy="0 0 0"/>
+          <geometry>
+            <mesh filename="${mesh_dir}/visual/finger.stl" scale="0.001 0.001 0.001"/>
+          </geometry>
+          <material name="grey"/>
+        </visual>
+      </link>
+      <!-- leftfinger -->
+      <joint name="${prefix}leftfinger_joint" type="prismatic">
+        <parent link="${prefix}link4"/>
+        <child link="${prefix}leftfinger"/>
+        <origin xyz="0 0 0.045" rpy="0 0 ${PI}"/>
+        <axis xyz="-1 0 0"/>
+        <limit
+          lower="0"
+          upper="0.0265"
+          effort="9.9"
+          velocity="9.9">
+        </limit>
+        <mimic joint="${prefix}gripper_joint" multiplier="0.024446"/>
+      </joint>
+      <link name="${prefix}leftfinger">
+        <collision>
+          <origin xyz="0 0 0" rpy="0 0 0"/>
+          <geometry>
+            <mesh filename="${mesh_dir}/collision/finger.stl" scale="0.001 0.001 0.001"/>
+          </geometry>
+        </collision>
+        <visual>
+          <origin xyz="0 0 0" rpy="0 0 0"/>
+          <geometry>
+            <mesh filename="${mesh_dir}/visual/finger.stl" scale="0.001 0.001 0.001"/>
+          </geometry>
+          <material name="grey"/>
+        </visual>
+      </link>
   </xacro:macro>
 </robot>

File: xavbot_moveit_config/config/xavbot.ros2_control.xacro (robot description, xacro)
@@ -36,4 +36,11 @@
                 <state_interface name="velocity"/>
             </joint>
+            <joint name="gripper_joint">
+                <command_interface name="position"/>
+                <state_interface name="position">
+                  <param name="initial_value">${initial_positions['gripper_joint']}</param>
+                </state_interface>
+                <state_interface name="velocity"/>
+            </joint>
         </ros2_control>
     </xacro:macro>

File: xavbot_moveit_config/config/xavbot.urdf.xacro (robot description, xacro)
@@ -5,5 +5,5 @@
     <xacro:include filename="$(find xavbot_description)/urdf/xavbot.arm.urdf.xacro" />
     <!-- Import control_xacro -->
-    <!-- <xacro:include filename="xavbot.ros2_control.xacro" />
-    <xacro:xavbot_ros2_control name="FakeSystem" initial_positions_file="$(arg initial_positions_file)"/> -->
+    <xacro:include filename="xavbot.ros2_control.xacro" />
+    <!-- <xacro:xavbot_ros2_control name="FakeSystem" initial_positions_file="$(arg initial_positions_file)"/> -->
 </robot>
