Commit message: Add second camera

File: xavbot_description/urdf/xavbot.platform.xacro (robot description, xacro)
@@ -17,5 +17,5 @@
       <origin xyz="${base_width / 2} ${base_length / 2} ${wheel_radius + 0.04}" rpy="0 0 0"/>
       <geometry>
-        <box size="0.25 0.25 0.08"/>
+        <box size="0.25 0.25 0.06"/>
       </geometry>
     </collision>

File: xavbot_description/urdf/xavbot.urdf.xacro (robot description, xacro)
@@ -7,6 +7,9 @@
   <xacro:xavbot_platform prefix="$(arg prefix)" mesh_dir="package://xavbot_description/meshes" />
   <xacro:include filename="$(find realsense2_description)/urdf/_d435i.urdf.xacro"/>
-  <xacro:sensor_d435i parent="base_link" use_nominal_extrinsics="false">
-    <origin xyz="0.03425 0.07 0.193" rpy="0 0 0"/>
+  <xacro:sensor_d435i parent="base_link" name="VIO_camera" use_nominal_extrinsics="false">
+    <origin xyz="0.17425 0.07 0.193" rpy="0 0 0"/>
+  </xacro:sensor_d435i>
+  <xacro:sensor_d435i parent="base_link" name="arm_camera" use_nominal_extrinsics="false">
+    <origin xyz="0.173 0.13 0.163" rpy="0 0.7854 0"/>
   </xacro:sensor_d435i>
   <!-- Import xavbot ros2_control description -->
