Commit message: Remove broken /odom publisher

File: xavbot_description/urdf/xavbot.urdf.xacro (robot description, xacro)
@@ -6,8 +6,7 @@
   <!-- Import Rviz colors -->
   <xacro:include filename="$(find xavbot_description)/urdf/xavbot.materials.xacro" />
-  <!-- Import diffbot ros2_control description -->
+  <!-- Import xavbot ros2_control description -->
   <xacro:include filename="$(find xavbot_description)/urdf/xavbot.ros2_control.xacro" />
   <xacro:xavbot prefix="$(arg prefix)" />
-  <xacro:xavbot_ros2_control
-    name="xavbot" prefix="$(arg prefix)" />
+  <xacro:xavbot_ros2_control name="xavbot" prefix="$(arg prefix)" />
 </robot>

File: xavbot_description/urdf/xavbot.xacro (robot description, xacro)
@@ -20,5 +20,5 @@
     </collision>
     <visual>
-      <origin xyz="0 0 0" rpy="0 0 0"/>
+      <origin xyz="0 0 0" rpy="0 0 ${PI}"/>
       <geometry>
         <mesh filename="package://xavbot_description/meshes/xavbot_chassis.stl" scale="0.001 0.001 0.001"/>
@@ -51,5 +51,5 @@
       </collision>
       <visual>
-        <origin xyz="0 0 0" rpy="${PI} 0 0"/>
+        <origin xyz="0 0 0" rpy="0 0 ${PI}"/>
         <geometry>
           <mesh filename="package://xavbot_description/meshes/d435.stl" scale="0.001 0.001 0.001"/>
@@ -61,5 +61,5 @@
       <parent link="${prefix}base_link"/>
       <child link="${prefix}camera_link"/>
-      <origin xyz="0.085 0 0.028" rpy="${PI} 0 0"/>
+      <origin xyz="0.085 0 0.028" rpy="0 0 0"/>
     </joint>
     <!-- front left wheel link -->

Commit message: Placeholder arm geometry and xacro tweaks

File: xavbot_description/urdf/xavbot.urdf.xacro (robot description, xacro)
@@ -4,9 +4,9 @@
   <!-- Import Geometry -->
   <xacro:include filename="$(find xavbot_description)/urdf/xavbot.xacro" />
+  <xacro:xavbot prefix="$(arg prefix)" mesh_dir="package://xavbot_description/meshes" />
   <!-- Import Rviz colors -->
   <xacro:include filename="$(find xavbot_description)/urdf/xavbot.materials.xacro" />
   <!-- Import xavbot ros2_control description -->
   <xacro:include filename="$(find xavbot_description)/urdf/xavbot.ros2_control.xacro" />
-  <xacro:xavbot prefix="$(arg prefix)" />
   <xacro:xavbot_ros2_control name="xavbot" prefix="$(arg prefix)" />
 </robot>

File: xavbot_description/urdf/xavbot.xacro (robot description, xacro)
@@ -1,5 +1,5 @@
 <?xml version="1.0"?>
 <robot xmlns:xacro="http://www.ros.org/wiki/xacro" name="xavbot">
-  <xacro:macro name="xavbot" params="prefix">
+  <xacro:macro name="xavbot" params="prefix='' mesh_dir='package://xavbot_description/meshes'">
   <!-- Constants for robot dimensions -->
   <xacro:property name="PI" value="3.1415926535897931"/>
@@ -23,5 +23,5 @@
       <origin xyz="0 0 ${wheel_radius}" rpy="0 0 0"/>
       <geometry>
-        <mesh filename="package://xavbot_description/meshes/visual/chassis.stl" scale="0.001 0.001 0.001"/>
+        <mesh filename="${mesh_dir}/visual/chassis.stl" scale="0.001 0.001 0.001"/>
       </geometry>
       <material name="grey"/>
@@ -48,5 +48,5 @@
         <origin xyz="0 0 0" rpy="0 0 0"/>
         <geometry>
-          <mesh filename="package://xavbot_description/meshes/collision/dummy_wheel.stl" scale="0.001 0.001 0.001"/>
+          <mesh filename="${mesh_dir}/collision/dummy_wheel.stl" scale="0.001 0.001 0.001"/>
         </geometry>
       </collision>
@@ -54,5 +54,5 @@
         <origin xyz="0 0 0" rpy="0 0 0"/>
         <geometry>
-          <mesh filename="package://xavbot_description/meshes/visual/dummy_wheel.stl" scale="0.001 0.001 0.001"/>
+          <mesh filename="${mesh_dir}/visual/dummy_wheel.stl" scale="0.001 0.001 0.001"/>
         </geometry>
         <material name="green"/>
@@ -79,5 +79,5 @@
         <origin xyz="0 0 0" rpy="0 0 0"/>
         <geometry>
-          <mesh filename="package://xavbot_description/meshes/collision/dummy_wheel.stl" scale="0.001 0.001 0.001"/>
+          <mesh filename="${mesh_dir}/collision/dummy_wheel.stl" scale="0.001 0.001 0.001"/>
         </geometry>
       </collision>
@@ -85,5 +85,5 @@
         <origin xyz="0 0 0" rpy="0 0 0"/>
         <geometry>
-          <mesh filename="package://xavbot_description/meshes/visual/dummy_wheel.stl" scale="0.001 0.001 0.001"/>
+          <mesh filename="${mesh_dir}/visual/dummy_wheel.stl" scale="0.001 0.001 0.001"/>
         </geometry>
         <material name="green"/>
@@ -110,11 +110,11 @@
           <origin xyz="0 0 0" rpy="0 0 0"/>
           <geometry>
-            <mesh filename="package://xavbot_description/meshes/collision/dummy_wheel.stl" scale="0.001 0.001 0.001"/>
-          </geometry>
-        </collision>
-        <visual>
-          <origin xyz="0 0 0" rpy="0 0 0"/>
-          <geometry>
-            <mesh filename="package://xavbot_description/meshes/visual/dummy_wheel.stl" scale="0.001 0.001 0.001"/>
+            <mesh filename="${mesh_dir}/collision/dummy_wheel.stl" scale="0.001 0.001 0.001"/>
+          </geometry>
+        </collision>
+        <visual>
+          <origin xyz="0 0 0" rpy="0 0 0"/>
+          <geometry>
+            <mesh filename="${mesh_dir}/visual/dummy_wheel.stl" scale="0.001 0.001 0.001"/>
           </geometry>
           <material name="green"/>
@@ -141,11 +141,11 @@
           <origin xyz="0 0 0" rpy="0 0 0"/>
           <geometry>
-            <mesh filename="package://xavbot_description/meshes/collision/dummy_wheel.stl" scale="0.001 0.001 0.001"/>
-          </geometry>
-        </collision>
-        <visual>
-          <origin xyz="0 0 0" rpy="0 0 0"/>
-          <geometry>
-            <mesh filename="package://xavbot_description/meshes/visual/dummy_wheel.stl" scale="0.001 0.001 0.001"/>
+            <mesh filename="${mesh_dir}/collision/dummy_wheel.stl" scale="0.001 0.001 0.001"/>
+          </geometry>
+        </collision>
+        <visual>
+          <origin xyz="0 0 0" rpy="0 0 0"/>
+          <geometry>
+            <mesh filename="${mesh_dir}/visual/dummy_wheel.stl" scale="0.001 0.001 0.001"/>
           </geometry>
           <material name="green"/>
@@ -174,10 +174,24 @@
         </limit>
       </joint>
-      <link name="${prefix}link0"/>
+      <link name="${prefix}link0">
+        <collision>
+          <origin xyz="0 0 0.05" rpy="0 0 0"/>
+          <geometry>
+            <box size="0.02 0.02 0.1"/>
+          </geometry>
+        </collision>
+        <visual>
+          <origin xyz="0 0 0.05" rpy="0 0 0"/>
+          <geometry>
+            <box size="0.02 0.02 0.1"/>
+          </geometry>
+          <material name="grey"/>
+        </visual>
+      </link>
       <!-- link1 -->
       <joint name="${prefix}link1_joint" type="revolute">
         <parent link="${prefix}link0"/>
         <child link="${prefix}link1"/>
-        <origin xyz="0 0 0.1" rpy="0 0 0"/>
+        <origin xyz="0 0 0.1" rpy="0 ${PI/2} 0"/>
         <axis xyz="0 1 0"/>
         <dynamics damping="0.2"/>
@@ -189,10 +203,24 @@
         </limit>
       </joint>
-      <link name="${prefix}link1"/>
+      <link name="${prefix}link1">
+        <collision>
+          <origin xyz="0 0 0.05" rpy="0 0 0"/>
+          <geometry>
+            <box size="0.02 0.02 0.1"/>
+          </geometry>
+        </collision>
+        <visual>
+          <origin xyz="0 0 0.05" rpy="0 0 0"/>
+          <geometry>
+            <box size="0.02 0.02 0.1"/>
+          </geometry>
+          <material name="grey"/>
+        </visual>
+      </link>
       <!-- link2 -->
       <joint name="${prefix}link2_joint" type="revolute">
         <parent link="${prefix}link1"/>
         <child link="${prefix}link2"/>
-        <origin xyz="0.1 0 0" rpy="0 ${PI/2} 0"/>
+        <origin xyz="0 0 0.1" rpy="0 ${PI/2} 0"/>
         <axis xyz="0 1 0"/>
         <dynamics damping="0.2"/>
@@ -204,10 +232,24 @@
         </limit>
       </joint>
-      <link name="${prefix}link2"/>
+      <link name="${prefix}link2">
+        <collision>
+          <origin xyz="0 0 0.015" rpy="0 0 0"/>
+          <geometry>
+            <box size="0.02 0.02 0.03"/>
+          </geometry>
+        </collision>
+        <visual>
+          <origin xyz="0 0 0.015" rpy="0 0 0"/>
+          <geometry>
+            <box size="0.02 0.02 0.03"/>
+          </geometry>
+          <material name="grey"/>
+        </visual>
+      </link>
       <!-- link3 -->
       <joint name="${prefix}link3_joint" type="fixed">
         <parent link="${prefix}link2"/>
         <child link="${prefix}link3"/>
-        <origin xyz="0.04 0 0" rpy="0 ${PI/2} 0"/>
+        <origin xyz="0 0 0.03" rpy="0 0 0"/>
         <axis xyz="0 0 1"/>
         <dynamics damping="0.2"/>

Commit message: Add realsense to urdf

File: xavbot_description/urdf/xavbot.urdf.xacro (robot description, xacro)
@@ -6,4 +6,8 @@
   <xacro:include filename="$(find xavbot_description)/urdf/xavbot.platform.xacro" />
   <xacro:xavbot_platform prefix="$(arg prefix)" mesh_dir="package://xavbot_description/meshes" />
+  <xacro:include filename="$(find realsense2_description)/urdf/_d435i.urdf.xacro"/>
+  <xacro:sensor_d435i parent="base_link" use_nominal_extrinsics="false">
+    <origin xyz="0.03425 0.07 0.193" rpy="0 0 0"/>
+  </xacro:sensor_d435i>
   <!-- Import xavbot ros2_control description -->
   <xacro:include filename="$(find xavbot_description)/urdf/xavbot.platform.ros2_control.xacro" />

Commit message: General improvements

File: xavbot_description/urdf/xavbot.urdf.xacro (robot description, xacro)
@@ -11,5 +11,5 @@
   </xacro:sensor_d435i>
   <xacro:sensor_d435i parent="base_link" name="arm_camera" use_nominal_extrinsics="false">
-    <origin xyz="0.173 0.13 0.163" rpy="0 0.7854 0"/>
+    <origin xyz="0.173 0.13 0.163" rpy="0 0.6981 0"/>
   </xacro:sensor_d435i>
   <!-- Import xavbot ros2_control description -->
